File: temperature-interface.sch (KiCad schematic (older format))
At the start: 25 parts, among them IC1 ATMEGA328-P, J1 USB_2, P1 1-Wire, P2 LCD, U1 MC34063, X1 16MHz

Commit message: value fix for the inductor at the boost converter
Parts:
- L1: value 50uH -> 180uH
Changed lines of the file:
@@
-EESchema Schematic File Version 2  date Fri 06 Jul 2012 03:26:37 AM CEST
+EESchema Schematic File Version 2  date Fri 06 Jul 2012 08:17:58 PM CEST
 LIBS:power
 LIBS:device
@@
 LIBS:contrib
 LIBS:valves
-EELAYER 43  0
+LIBS:temperature-interface-cache
+EELAYER 25  0
 EELAYER END
 $Descr A4 11700 8267
@@
 P 9600 4950
 F 0 "L1" V 9550 4950 40  0000 C CNN
-F 1 "50uH" V 9700 4950 40  0000 C CNN
+F 1 "180uH" V 9700 4950 40  0000 C CNN
 	1    9600 4950
 	1    0    0    -1
